File: hw/iqdemod.sch (EAGLE design)
At the start: 54 parts, among them U1 AD8348, X1 SMA-142-0701-881/886, X10 SMA-142-0701-881/886, X11 SMA-142-0701-881/886, X12 SMA-142-0701-881/886, X2 SMA-142-0701-881/886, X3 SMA-142-0701-881/886, X4 VGIN, X5 VGIN, X9 SMA-142-0701-881/886

Commit message: implement new baseband filter topology and add pad for supply
Parts:
- removed C14, C15: (no value), rcl:C-EUC0603
- added X6: VIN, wirepad:SMD2
- C11: value (none) -> 10u
- C13: value (none) -> 1u
- X5: value VGIN -> EN
Connections:
- net +5V: now also C11.1, C13.1, X6.P
- net GND: now also C11.2, C13.2
- net N$11: no longer C11.1, C9.1
- net N$12: no longer C13.1, C15.1
- net N$16: no longer C10.1, C9.2
- net N$17: now also C10.1; no longer C10.2
- net N$27: no longer C13.2, C14.1
- net N$28: now also C9.1; no longer C14.2
- net VREF: now also C10.2, C9.2; no longer C11.2, C15.2
Other:
- note added: "Rev.:1"
- note removed: "Rev.:0"
- note removed: "todo: calculate 1MHz baseband lowpass filter"
- moved on the sheet: C10, C11, C12, C13, C16, C9, L1, L2, L3, L4, R10, R11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

Commit message: rev. 1: finished board
Connections:
- net +5V: no longer U1M.ENVG
- net N$30: now also U1M.ENVG
Other:
- moved on the sheet: FB1, FB2, FB3, R14, R3, R5, X4, X5
